Commit message: added right caster wheel support

File: my_rb1_description/urdf/my_rb1_robot.urdf (robot description, URDF)
Before this commit: robot my_rb1_robot, 7 links, 6 joints
Links:
- link back_caster: geometry collision sphere radius=0.025; collision sphere radius=0.065
- link front_caster: geometry collision sphere radius=0.025; collision sphere radius=0.065
Joints:
- joint joint_base_caster_wheel_back: origin xyz=-0.1 0.0 -0.15 rpy=0 0 0 -> xyz=-0.1 0.0 -0.10 rpy=0 0 0
- joint joint_base_caster_wheel_front: origin xyz=0.1 0.0 -0.15 rpy=0 0 0 -> xyz=0.1 0.0 -0.10 rpy=0 0 0
